Commit message: Update my-robot.xacro

File: src/funny_3dof_robot/robot/visual/my-robot.xacro (robot description, xacro)
@@ -12,9 +12,9 @@
         <parent link="link_0"/>
         <child link="link_1"/>
-        <origin xyz="0 0 0"/>
+        <origin xyz="0 0 0.2"/>
     </joint>
     <link name="link_1">
     <visual>
-        <origin rpy="0 0 0" xyz="0 0 0.2"/>
+        <origin rpy="0 0 0" xyz="0 0 0"/>
         <geometry>
         <mesh filename="package://funny_3dof_robot/meshes/link_1.stl"/>
@@ -25,11 +25,11 @@
         <parent link="link_1"/>
         <child link="link_2"/>
-        <axis xyz="0 1 0"/>
+        <axis xyz="0 0 1"/>
         <limit effort="100.0" lower="-1.57" upper="1.57" velocity="1.0"/>
-        <origin xyz="0 0 0.2"/>
+        <origin rpy="-1.57075 -1.57075  0" xyz="0 -0.12 0"/>
     </joint>
     <link name="link_2">
     <visual>
-        <origin rpy="-1.57075 -1.57075  0" xyz="0 -0.12 0"/>
+        <origin rpy="0 0 0" xyz="0 0 0"/>
         <geometry>
         <mesh filename="package://funny_3dof_robot/meshes/link_2.stl"/>
@@ -42,9 +42,9 @@
         <axis xyz="0 0 1"/>
         <limit effort="100.0" lower="-1.57" upper="1.57" velocity="1.0"/>
-        <origin rpy="-1.57075 -1.57075  0" xyz="0 -0.12 0.25"/>
+        <origin rpy="0 0 0" xyz="0.25 0 0.1"/>
     </joint>
     <link name="link_3">
     <visual>
-        <origin rpy="0 0 0" xyz="0 0 0.1"/>
+        <origin rpy="0 0 0" xyz="0 0 0"/>
         <geometry>
         <mesh filename="package://funny_3dof_robot/meshes/link_3.stl"/>
@@ -57,5 +57,5 @@
         <axis xyz="0 0 1"/>
         <limit effort="100.0" lower="-1.57" upper="1.57" velocity="1.0"/>
-        <origin rpy="0 1.57 0" xyz="0.28 0 0.1"/>
+        <origin rpy="1.57 0 1.57" xyz="0.28 0 0"/>
     </joint>
     <link name="end_effector">

Commit message: ucpdate xacro

File: src/funny_3dof_robot/robot/visual/my-robot.xacro (robot description, xacro)
@@ -1,4 +1,4 @@
 <?xml version="1.0"?>
-<robot xmlns:xacro="http://www.ros.org/wiki/xacro" name="example">
+<robot xmlns:xacro="http://www.ros.org/wiki/xacro" name="3DOF_Robot">
     <link name="link_0">
     <visual>
@@ -9,7 +9,8 @@
     </visual>
     </link>
-    <joint name="joint_0" type="fixed">
+    <joint name="joint_0" type="continuous">
         <parent link="link_0"/>
         <child link="link_1"/>
+        <axis xyz="0 0 1"/>
         <origin xyz="0 0 0.2"/>
     </joint>
@@ -26,5 +27,5 @@
         <child link="link_2"/>
         <axis xyz="0 0 1"/>
-        <limit effort="100.0" lower="-1.57" upper="1.57" velocity="1.0"/>
+        <limit effort="100.0" lower="-3.14" upper="3.14" velocity="1.0"/>
         <origin rpy="-1.57075 -1.57075  0" xyz="0 -0.12 0"/>
     </joint>
@@ -41,5 +42,5 @@
         <child link="link_3"/>
         <axis xyz="0 0 1"/>
-        <limit effort="100.0" lower="-1.57" upper="1.57" velocity="1.0"/>
+        <limit effort="100.0" lower="-3.14" upper="3.14" velocity="1.0"/>
         <origin rpy="0 0 0" xyz="0.25 0 0.1"/>
     </joint>
@@ -56,5 +57,5 @@
         <child link="end_effector"/>
         <axis xyz="0 0 1"/>
-        <limit effort="100.0" lower="-1.57" upper="1.57" velocity="1.0"/>
+        <limit effort="100.0" lower="-3.14" upper="3.14" velocity="1.0"/>
         <origin rpy="1.57 0 1.57" xyz="0.28 0 0"/>
     </joint>

Commit message: random and rvizconfig

File: src/funny_3dof_robot/robot/visual/my-robot.xacro (robot description, xacro)
@@ -53,9 +53,9 @@
     </visual>
     </link>
-    <joint name="joint_3" type="revolute">
+    <joint name="joint_3" type="fixed">
         <parent link="link_3"/>
         <child link="end_effector"/>
         <axis xyz="0 0 1"/>
-        <limit effort="100.0" lower="-3.14" upper="3.14" velocity="1.0"/>
+        <!-- <limit effort="100.0" lower="-3.14" upper="3.14" velocity="1.0"/> -->
         <origin rpy="1.57 0 1.57" xyz="0.28 0 0"/>
     </joint>
